File: src/pcb/dacboard/header.kicad_sch (KiCad schematic)
At the start: 1 part, among them J4 Conn_01x24_Socket

Commit message: dacboard routing
Parts:
- removed J4: Conn_01x24_Socket, symbol Connector:Conn_01x24_Socket
