File: src/pcb/dacboard/dacboard.kicad_pcb (KiCad board)
At the start: 12 copper layers, 284 parts, among them J1 Screw_Terminal_01x03, J10 Conn_02x17_Odd_Even, J11 Conn_02x17_Odd_Even, J12 Conn_02x12_Odd_Even, J13 Conn_02x12_Odd_Even, J14 Conn_01x14, J15 Conn_01x14, J16 Conn_02x17_Odd_Even, J17 Conn_01x14, J18 Conn_01x14, J19 Conn_01x14, J2 Screw_Terminal_01x02, J20 Conn_01x14, J21 Conn_01x14, J22 Conn_01x06, J3 Conn_01x30_Socket, J4 Conn_01x14, J5 Conn_02x12_Odd_Even, J6 Conn_01x14, J7 Conn_02x06_Odd_Even, J8 Conn_02x06_Odd_Even, J9 Conn_02x17_Odd_Even, U1 LTC6655CHMS8-2.5_PBF, U10 AD5791BRUZ, U100 ISO6761FQDWRQ1, U101 ISO6761FQDWRQ1, U102 ISO6761FQDWRQ1, U103 ISO6761FQDWRQ1, U104 ISO6761FQDWRQ1, U105 ISO6761FQDWRQ1, U11 AD8676xR, U12 AD8676xR, U13 AD5791BRUZ, U14 AD8676xR, U15 AD5791BRUZ, U16 AD8676xR, U17 AD5791BRUZ, U18 AD8676xR, U19 AD5791BRUZ, U2 LTC6655CHMS8-2.5_PBF, U20 AD8676xR, U21 AD5791BRUZ, U22 AD8676xR, U23 AD8676xR, U24 AD8676xR, U25 AD8676xR, U26 AD5791BRUZ, U27 AD5791BRUZ, U28 AD5791BRUZ, U29 AD5791BRUZ, U3 LTC6655CHMS8-2.5_PBF, U30 AD8676xR, U31 AD8676xR, U32 AD5791BRUZ, U33 AD5791BRUZ, U34 AD8676xR, U35 AD8676xR, U36 AD8676xR, U37 AD8676xR, U38 AD5791BRUZ, U39 AD5791BRUZ, U4 LTC6655CHMS8-2.5_PBF, U40 AD5791BRUZ, U41 AD5791BRUZ, U42 AD8676xR, U43 AD8676xR, U44 AD5791BRUZ, U45 AD5791BRUZ, U46 AD8676xR, U47 AD8676xR, U48 AD8676xR, U49 AD8676xR, U5 LTC6655CHMS8-2.5_PBF, U50 AD5791BRUZ, U51 AD5791BRUZ, U52 AD5791BRUZ, U53 AD5791BRUZ, U54 AD8676xR, U55 AD8676xR, U56 AD5791BRUZ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

Commit message: analog side layout
Parts:
- moved R15 127.3 mm to (162.7, 83.3), turned to -45 degrees
- moved R40 126.2 mm to (159.5, 86.5), turned to -45 degrees
- moved R14 80.4 mm to (27.0, 121.0), turned to 90 degrees
- moved R13 75.8 mm to (27.0, 126.1), turned to 90 degrees
- moved C21 59.6 mm to (30.9, 121.0)
- moved C17 58.5 mm to (40.0, 182.0), turned to -90 degrees
- moved C13 57.6 mm to (25.0, 175.5), turned to -90 degrees
- moved C20 55.7 mm to (30.9, 126.0)
- moved C9 55.4 mm to (25.0, 165.5), turned to -90 degrees
- moved C5 53.8 mm to (25.0, 155.5), turned to -90 degrees
- moved C1 52.8 mm to (25.0, 145.5), turned to -90 degrees
- moved R11 45.5 mm to (55.0, 133.0)
- moved C14 43.8 mm to (35.0, 176.0), turned to -90 degrees
- moved R12 43.7 mm to (59.9, 133.0)
- moved C10 41.7 mm to (35.0, 166.0), turned to -90 degrees
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Connections:
- C17 pad 1: Net-(U9B-+) -> Net-(U9A-+)
- R1 pad 2: Net-(U9B-+) -> Net-(U9A-+)
- R10 pad 1: Net-(U9B--) -> Net-(U9A--)
- R10 pad 2: Net-(U9B--) -> Net-(U9A--)
- R2 pad 2: Net-(U9B-+) -> Net-(U9A-+)
- R3 pad 2: Net-(U9B-+) -> Net-(U9A-+)
- R4 pad 2: Net-(U9B-+) -> Net-(U9A-+)
- R5 pad 2: Net-(U9B-+) -> Net-(U9A-+)
- R6 pad 2: Net-(U9B-+) -> Net-(U9A-+)
- R7 pad 2: Net-(U9B-+) -> Net-(U9A-+)
- R8 pad 2: Net-(U9B-+) -> Net-(U9A-+)
- R9 pad 1: Net-(U9A--) -> Net-(U9B--)
- R9 pad 2: Net-(U9A--) -> Net-(U9B--)
- R9 pad 3: Net-(U9A--) -> Net-(U9B--)
- R9 pad 6: Net-(U9B-+) -> Net-(U9A-+)
- R9 pad 7: Net-(U9B-+) -> Net-(U9A-+)
- U9 pad 1: Net-(R11-Pad1) -> Net-(R10-Pad8)
- U9 pad 3: AGND -> Net-(U9A-+)
- U9 pad 5: Net-(U9B-+) -> AGND
- U9 pad 7: Net-(R10-Pad8) -> Net-(R11-Pad1)
Routing:
- net AGND: track 4.62 -> 324.8 mm, vias 4 -> 88
- net VREF+: track 57.6 -> 248.9 mm, vias 24 -> 50
- net VDD: track 69.2 -> 259.0 mm, vias 30 -> 118
- net +5VD: track 1.00 -> 105.8 mm, vias 0 -> 48
- net DGND: track 22.5 -> 123.9 mm, vias 16 -> 96
- net Net-(U9A-+): track 0.00 -> 83.8 mm
- net VSS: track 120.6 -> 194.6 mm, vias 76 -> 146
- net Net-(R11-Pad1): track 0.00 -> 26.0 mm
- net Net-(R10-Pad8): track 0.00 -> 18.8 mm
- net Net-(U9A--): track 0.00 -> 14.6 mm
- net Net-(U9B--): track 0.00 -> 13.3 mm
- net VOUT_F6: track 0.00 -> 8.97 mm
- net VOUT_F5: track 0.00 -> 8.97 mm
- net VOUT_F2: track 0.00 -> 8.97 mm
- net VOUT_F8: track 0.00 -> 8.97 mm
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
Commit message: pcb should reroute
Parts:
- moved C35 89.7 mm to (-28.7, 47.8)
- moved C36 78.5 mm to (7.50, 18.3)
- moved C24 77.0 mm to (5.50, 30.8)
- moved C23 70.5 mm to (-9.50, 45.5)
- moved C22 28.1 mm to (13.0, 48.7)
- moved C34 25.8 mm to (15.5, 49.9)
- moved C33 15.1 mm to (266.0, 60.2), turned to 0 degrees
- moved U10 15.0 mm to (46.0, 55.0)
- moved U13 15.0 mm to (66.0, 55.0)
- moved U15 15.0 mm to (86.0, 55.0)
- moved U17 15.0 mm to (106.0, 55.0)
- moved U19 15.0 mm to (126.0, 55.0)
- moved U21 15.0 mm to (146.0, 55.0)
- moved U26 15.0 mm to (166.0, 55.0)
- moved U27 15.0 mm to (186.0, 55.0)
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Routing:
- net CLR_N: track 899.3 -> 277.8 mm, vias 26 -> 2
- net RESET_N: track 909.1 -> 304.0 mm, vias 26 -> 2
- net VREF+: track 248.9 -> 6.47 mm, vias 50 -> 2
- net VSS: track 194.6 -> 2.73 mm, vias 146 -> 2
- net VDD: track 259.0 -> 87.9 mm, vias 118 -> 18
- net DGND: track 123.9 -> 0.00 mm, vias 96 -> 0
- net AGND: track 324.8 -> 203.1 mm, vias 88 -> 40
- net BUF12_VOUT: track 107.8 -> 0.00 mm
- net +5VD: track 105.8 -> 0.00 mm, vias 48 -> 0
- net BUF11_VOUT: track 91.0 -> 0.00 mm
- net BUF13_VOUT: track 87.6 -> 0.00 mm
- net BUF24_VOUT: track 87.5 -> 0.00 mm
- net BUF10_VOUT: track 76.1 -> 0.00 mm
- net DAC6_SYNC_N: track 80.0 -> 6.82 mm
- net BUF23_VOUT: track 72.6 -> 0.00 mm
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