File: src/pcb/dacboard/dacboard.kicad_pcb (KiCad board)
At the start: 14 copper layers, 338 parts, among them J1 Screw_Terminal_01x03, J10 Conn_02x17_Odd_Even, J11 Conn_02x17_Odd_Even, J12 Conn_02x12_Odd_Even, J13 Conn_02x12_Odd_Even, J14 Conn_01x14, J15 Conn_01x14, J16 Conn_02x17_Odd_Even, J17 Conn_01x14, J18 Conn_01x14, J19 Conn_01x14, J2 Screw_Terminal_01x02, J20 Conn_01x14, J21 Conn_01x14, J22 Conn_01x06, J23 Conn_01x05, J24 Conn_01x03, J25 Conn_01x02, J3 Conn_01x30_Socket, J4 Conn_01x14, J5 Conn_02x12_Odd_Even, J6 Conn_01x14, J7 Conn_02x06_Odd_Even, J8 Conn_02x06_Odd_Even, J9 Conn_02x17_Odd_Even, U1 LTC6655CHMS8-2.5_PBF, U10 AD5791BRUZ, U100 ISO6761FQDWRQ1, U101 ISO6761FQDWRQ1, U102 ISO6761FQDWRQ1, U103 ISO6761FQDWRQ1, U104 ISO6761FQDWRQ1, U105 ISO6761FQDWRQ1, U11 AD8676xR, U12 AD8676xR, U13 AD5791BRUZ, U14 AD8676xR, U15 AD5791BRUZ, U16 AD8676xR, U17 AD5791BRUZ, U18 AD8676xR, U19 AD5791BRUZ, U2 LTC6655CHMS8-2.5_PBF, U20 AD8676xR, U21 AD5791BRUZ, U22 AD8676xR, U23 AD8676xR, U24 AD8676xR, U25 AD8676xR, U26 AD5791BRUZ, U27 AD5791BRUZ, U28 AD5791BRUZ, U29 AD5791BRUZ, U3 LTC6655CHMS8-2.5_PBF, U30 AD8676xR, U31 AD8676xR, U32 AD5791BRUZ, U33 AD5791BRUZ, U34 AD8676xR, U35 AD8676xR, U36 AD8676xR, U37 AD8676xR, U38 AD5791BRUZ, U39 AD5791BRUZ, U4 LTC6655CHMS8-2.5_PBF, U40 AD5791BRUZ, U41 AD5791BRUZ, U42 AD8676xR, U43 AD8676xR, U44 AD5791BRUZ, U45 AD5791BRUZ, U46 AD8676xR, U47 AD8676xR, U48 AD8676xR, U49 AD8676xR, U5 LTC6655CHMS8-2.5_PBF, U50 AD5791BRUZ, U51 AD5791BRUZ, U52 AD5791BRUZ, U53 AD5791BRUZ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

Commit message: more capacitors
Parts:
- added REF**: C_0402_1005Metric_Pad0.74x0.62mm_HandSolder, Capacitor_SMD:C_0402_1005Metric_Pad0.74x0.62mm_HandSolder, F.Cu at (171.6, 40.2)
- added REF**: C_0402_1005Metric_Pad0.74x0.62mm_HandSolder, Capacitor_SMD:C_0402_1005Metric_Pad0.74x0.62mm_HandSolder, F.Cu at (265.1, 34.6)
- added REF**: C_0402_1005Metric_Pad0.74x0.62mm_HandSolder, Capacitor_SMD:C_0402_1005Metric_Pad0.74x0.62mm_HandSolder, F.Cu at (111.5, 40.2)
- added REF**: C_0402_1005Metric_Pad0.74x0.62mm_HandSolder, Capacitor_SMD:C_0402_1005Metric_Pad0.74x0.62mm_HandSolder, F.Cu at (191.6, 40.2)
- added REF**: C_0402_1005Metric_Pad0.74x0.62mm_HandSolder, Capacitor_SMD:C_0402_1005Metric_Pad0.74x0.62mm_HandSolder, F.Cu at (105.1, 34.6)
- added REF**: C_0402_1005Metric_Pad0.74x0.62mm_HandSolder, Capacitor_SMD:C_0402_1005Metric_Pad0.74x0.62mm_HandSolder, F.Cu at (91.5, 40.2)
- added REF**: C_0402_1005Metric_Pad0.74x0.62mm_HandSolder, Capacitor_SMD:C_0402_1005Metric_Pad0.74x0.62mm_HandSolder, F.Cu at (185.1, 34.6)
- added REF**: C_0402_1005Metric_Pad0.74x0.62mm_HandSolder, Capacitor_SMD:C_0402_1005Metric_Pad0.74x0.62mm_HandSolder, F.Cu at (231.6, 40.2)
- added REF**: C_0402_1005Metric_Pad0.74x0.62mm_HandSolder, Capacitor_SMD:C_0402_1005Metric_Pad0.74x0.62mm_HandSolder, F.Cu at (151.6, 40.2)
- added REF**: C_0402_1005Metric_Pad0.74x0.62mm_HandSolder, Capacitor_SMD:C_0402_1005Metric_Pad0.74x0.62mm_HandSolder, F.Cu at (31.6, 40.2)
- added REF**: C_0402_1005Metric_Pad0.74x0.62mm_HandSolder, Capacitor_SMD:C_0402_1005Metric_Pad0.74x0.62mm_HandSolder, F.Cu at (145.1, 34.6)
- added REF**: C_0402_1005Metric_Pad0.74x0.62mm_HandSolder, Capacitor_SMD:C_0402_1005Metric_Pad0.74x0.62mm_HandSolder, F.Cu at (165.1, 34.6)
- added REF**: C_0402_1005Metric_Pad0.74x0.62mm_HandSolder, Capacitor_SMD:C_0402_1005Metric_Pad0.74x0.62mm_HandSolder, F.Cu at (251.6, 40.2)
- added REF**: C_0402_1005Metric_Pad0.74x0.62mm_HandSolder, Capacitor_SMD:C_0402_1005Metric_Pad0.74x0.62mm_HandSolder, F.Cu at (211.6, 40.2)
- added REF**: C_0402_1005Metric_Pad0.74x0.62mm_HandSolder, Capacitor_SMD:C_0402_1005Metric_Pad0.74x0.62mm_HandSolder, F.Cu at (225.1, 34.6)
- added REF**: C_0402_1005Metric_Pad0.74x0.62mm_HandSolder, Capacitor_SMD:C_0402_1005Metric_Pad0.74x0.62mm_HandSolder, F.Cu at (85.1, 34.6)
- added REF**: C_0402_1005Metric_Pad0.74x0.62mm_HandSolder, Capacitor_SMD:C_0402_1005Metric_Pad0.74x0.62mm_HandSolder, F.Cu at (245.1, 34.6)
- added REF**: C_0402_1005Metric_Pad0.74x0.62mm_HandSolder, Capacitor_SMD:C_0402_1005Metric_Pad0.74x0.62mm_HandSolder, F.Cu at (125.1, 34.6)
- added REF**: C_0402_1005Metric_Pad0.74x0.62mm_HandSolder, Capacitor_SMD:C_0402_1005Metric_Pad0.74x0.62mm_HandSolder, B.Cu at (244.4, 40.2)
- added REF**: C_0402_1005Metric_Pad0.74x0.62mm_HandSolder, Capacitor_SMD:C_0402_1005Metric_Pad0.74x0.62mm_HandSolder, B.Cu at (70.9, 34.6)
- added REF**: C_0402_1005Metric_Pad0.74x0.62mm_HandSolder, Capacitor_SMD:C_0402_1005Metric_Pad0.74x0.62mm_HandSolder, F.Cu at (45.1, 34.6)
- added REF**: C_0402_1005Metric_Pad0.74x0.62mm_HandSolder, Capacitor_SMD:C_0402_1005Metric_Pad0.74x0.62mm_HandSolder, B.Cu at (124.5, 40.2)
- added REF**: C_0402_1005Metric_Pad0.74x0.62mm_HandSolder, Capacitor_SMD:C_0402_1005Metric_Pad0.74x0.62mm_HandSolder, B.Cu at (150.9, 34.6)
- added REF**: C_0402_1005Metric_Pad0.74x0.62mm_HandSolder, Capacitor_SMD:C_0402_1005Metric_Pad0.74x0.62mm_HandSolder, B.Cu at (30.9, 34.6)
- added REF**: C_0402_1005Metric_Pad0.74x0.62mm_HandSolder, Capacitor_SMD:C_0402_1005Metric_Pad0.74x0.62mm_HandSolder, B.Cu at (184.4, 40.2)
- added REF**: C_0402_1005Metric_Pad0.74x0.62mm_HandSolder, Capacitor_SMD:C_0402_1005Metric_Pad0.74x0.62mm_HandSolder, B.Cu at (204.4, 40.2)
- added REF**: C_0402_1005Metric_Pad0.74x0.62mm_HandSolder, Capacitor_SMD:C_0402_1005Metric_Pad0.74x0.62mm_HandSolder, B.Cu at (210.9, 34.6)
- added REF**: C_0402_1005Metric_Pad0.74x0.62mm_HandSolder, Capacitor_SMD:C_0402_1005Metric_Pad0.74x0.62mm_HandSolder, B.Cu at (64.5, 40.2)
- added REF**: C_0402_1005Metric_Pad0.74x0.62mm_HandSolder, Capacitor_SMD:C_0402_1005Metric_Pad0.74x0.62mm_HandSolder, B.Cu at (224.4, 40.2)
- added REF**: C_0402_1005Metric_Pad0.74x0.62mm_HandSolder, Capacitor_SMD:C_0402_1005Metric_Pad0.74x0.62mm_HandSolder, B.Cu at (170.9, 34.6)
- added REF**: C_0402_1005Metric_Pad0.74x0.62mm_HandSolder, Capacitor_SMD:C_0402_1005Metric_Pad0.74x0.62mm_HandSolder, B.Cu at (84.5, 40.2)
- added REF**: C_0402_1005Metric_Pad0.74x0.62mm_HandSolder, Capacitor_SMD:C_0402_1005Metric_Pad0.74x0.62mm_HandSolder, F.Cu at (131.6, 40.2)
- added REF**: C_0402_1005Metric_Pad0.74x0.62mm_HandSolder, Capacitor_SMD:C_0402_1005Metric_Pad0.74x0.62mm_HandSolder, B.Cu at (264.4, 40.2)
- added REF**: C_0402_1005Metric_Pad0.74x0.62mm_HandSolder, Capacitor_SMD:C_0402_1005Metric_Pad0.74x0.62mm_HandSolder, B.Cu at (164.4, 40.2)
- added REF**: C_0402_1005Metric_Pad0.74x0.62mm_HandSolder, Capacitor_SMD:C_0402_1005Metric_Pad0.74x0.62mm_HandSolder, B.Cu at (90.9, 34.6)
- added REF**: C_0402_1005Metric_Pad0.74x0.62mm_HandSolder, Capacitor_SMD:C_0402_1005Metric_Pad0.74x0.62mm_HandSolder, B.Cu at (110.9, 34.6)
- added REF**: C_0402_1005Metric_Pad0.74x0.62mm_HandSolder, Capacitor_SMD:C_0402_1005Metric_Pad0.74x0.62mm_HandSolder, B.Cu at (50.9, 34.6)
- added REF**: C_0402_1005Metric_Pad0.74x0.62mm_HandSolder, Capacitor_SMD:C_0402_1005Metric_Pad0.74x0.62mm_HandSolder, B.Cu at (250.9, 34.6)
- added REF**: C_0402_1005Metric_Pad0.74x0.62mm_HandSolder, Capacitor_SMD:C_0402_1005Metric_Pad0.74x0.62mm_HandSolder, B.Cu at (104.5, 40.2)
- added REF**: C_0402_1005Metric_Pad0.74x0.62mm_HandSolder, Capacitor_SMD:C_0402_1005Metric_Pad0.74x0.62mm_HandSolder, B.Cu at (130.9, 34.6)
- added REF**: C_0402_1005Metric_Pad0.74x0.62mm_HandSolder, Capacitor_SMD:C_0402_1005Metric_Pad0.74x0.62mm_HandSolder, B.Cu at (144.4, 40.2)
- added REF**: C_0402_1005Metric_Pad0.74x0.62mm_HandSolder, Capacitor_SMD:C_0402_1005Metric_Pad0.74x0.62mm_HandSolder, B.Cu at (44.5, 40.2)
- added REF**: C_0402_1005Metric_Pad0.74x0.62mm_HandSolder, Capacitor_SMD:C_0402_1005Metric_Pad0.74x0.62mm_HandSolder, F.Cu at (51.5, 40.2)
- added REF**: C_0402_1005Metric_Pad0.74x0.62mm_HandSolder, Capacitor_SMD:C_0402_1005Metric_Pad0.74x0.62mm_HandSolder, B.Cu at (190.9, 34.6)
- added REF**: C_0402_1005Metric_Pad0.74x0.62mm_HandSolder, Capacitor_SMD:C_0402_1005Metric_Pad0.74x0.62mm_HandSolder, B.Cu at (230.9, 34.6)
- added REF**: C_0402_1005Metric_Pad0.74x0.62mm_HandSolder, Capacitor_SMD:C_0402_1005Metric_Pad0.74x0.62mm_HandSolder, F.Cu at (205.1, 34.6)
- added REF**: C_0402_1005Metric_Pad0.74x0.62mm_HandSolder, Capacitor_SMD:C_0402_1005Metric_Pad0.74x0.62mm_HandSolder, F.Cu at (65.1, 34.6)
- added REF**: C_0402_1005Metric_Pad0.74x0.62mm_HandSolder, Capacitor_SMD:C_0402_1005Metric_Pad0.74x0.62mm_HandSolder, F.Cu at (71.5, 40.2)
Routing:
- net AGND: vias 183 -> 231
