File: src/pcb/dacboard/dacboard.kicad_pcb (KiCad board)
At the start: 14 copper layers, 273 x 186 mm, 387 parts, among them J1 Screw_Terminal_01x03, J10 Conn_02x17_Odd_Even, J11 Conn_02x17_Odd_Even, J12 Conn_02x12_Odd_Even, J13 Conn_02x12_Odd_Even, J14 Conn_01x14, J15 Conn_01x14, J16 Conn_02x17_Odd_Even, J17 Conn_01x14, J18 Conn_01x14, J19 Conn_01x14, J2 Screw_Terminal_01x02, J20 Conn_01x14, J21 Conn_01x14, J23 Conn_01x05, J24 Conn_01x03, J25 Conn_01x02, J26 Screw_Terminal_01x02, J3 Conn_01x30_Socket, J4 Conn_01x14, J5 Conn_02x12_Odd_Even, J6 Conn_01x14, J7 Conn_02x06_Odd_Even, J8 Conn_02x06_Odd_Even, J9 Conn_02x17_Odd_Even, U1 LTC6655CHMS8-2.5_PBF, U10 AD5791BRUZ, U100 ISO6761FQDWRQ1, U101 ISO6761FQDWRQ1, U102 ISO6761FQDWRQ1, U103 ISO6761FQDWRQ1, U104 ISO6761FQDWRQ1, U105 ISO6761FQDWRQ1, U11 AD8676xR, U12 AD8676xR, U13 AD5791BRUZ, U14 AD8676xR, U15 AD5791BRUZ, U16 AD8676xR, U17 AD5791BRUZ, U18 AD8676xR, U19 AD5791BRUZ, U2 LTC6655CHMS8-2.5_PBF, U20 AD8676xR, U21 AD5791BRUZ, U22 AD8676xR, U23 AD8676xR, U24 AD8676xR, U25 AD8676xR, U26 AD5791BRUZ, U27 AD5791BRUZ, U28 AD5791BRUZ, U29 AD5791BRUZ, U3 LTC6655CHMS8-2.5_PBF, U30 AD8676xR, U31 AD8676xR, U32 AD5791BRUZ, U33 AD5791BRUZ, U34 AD8676xR, U35 AD8676xR, U36 AD8676xR, U37 AD8676xR, U38 AD5791BRUZ, U39 AD5791BRUZ, U4 LTC6655CHMS8-2.5_PBF, U40 AD5791BRUZ, U41 AD5791BRUZ, U42 AD8676xR, U43 AD8676xR, U44 AD5791BRUZ, U45 AD5791BRUZ, U46 AD8676xR, U47 AD8676xR, U48 AD8676xR, U49 AD8676xR, U5 LTC6655CHMS8-2.5_PBF, U50 AD5791BRUZ, U51 AD5791BRUZ, U52 AD5791BRUZ, U53 AD5791BRUZ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

Commit message: board name and date
Other:
- board text added: "Sigillito/Shize DAC V4.0 12/01/2025"
Changed lines of the file:
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@@
+		)
+	)
+	(gr_text "Sigillito/Shize DAC V4.0\n12/01/2025"
+		(at 26.18 192.92 0)
+		(layer "F.SilkS")
+		(effects
+			(font
+				(size 1 1)
+				(thickness 0.1)
+			)
+			(justify left bottom)
 		)
 	)
