File: src/pcb/dacboard/isolator13-18.kicad_sch (KiCad schematic)
At the start: 18 parts, among them U100 ISO7761FQDBQRQ1, U95 ISO7761FQDBQRQ1, U96 ISO7761FQDBQRQ1, U97 ISO7761FQDBQRQ1, U98 ISO7761FQDBQRQ1, U99 ISO7761FQDBQRQ1

Commit message: dacboard routing
Parts:
- removed U100, U95, U96, U97, U98, U99: ISO7761FQDBQRQ1, DBQ16_TEX, symbol 2025-11-18_20-36-36:ISO7761FQDBQRQ1
- added U94, U95, U96, U97, U98, U99: ISO6761FQDWRQ1, ISO6761:SOIC16_DW_TEX, symbol 2025-11-20_00-47-15:ISO6761FQDWRQ1
- C100, C101, C102, C103, C104, C105, C106, C107, C96, C97, C98, C99: footprint (none) -> Capacitor_SMD:C_0402_1005Metric_Pad0.74x0.62mm_HandSolder
Connections:
- net +5VD: now also U94.16 (VCC2), U95.16 (VCC2), U96.16 (VCC2), U97.16 (VCC2), U98.16 (VCC2), U99.16 (VCC2)
- net CS_N_CH13: now also U94.5 (IND)
- net CS_N_CH14: now also U95.5 (IND)
- net CS_N_CH15: now also U96.5 (IND)
- net CS_N_CH16: now also U97.5 (IND)
- net CS_N_CH17: now also U98.5 (IND)
- net CS_N_CH18: now also U99.5 (IND)
- net DAC13_LDAC_N: now also U94.15 (OUTA)
- net DAC13_SCLK: now also U94.13 (OUTC)
- net DAC13_SDIN: now also U94.14 (OUTB)
- net DAC13_SDO: now also U94.10 (INF)
- net DAC13_SYNC_N: now also U94.12 (OUTD)
- net DAC14_LDAC_N: now also U95.15 (OUTA)
- net DAC14_SCLK: now also U95.13 (OUTC)
- net DAC14_SDIN: now also U95.14 (OUTB)
- net DAC14_SDO: now also U95.10 (INF)
- net DAC14_SYNC_N: now also U95.12 (OUTD)
- net DAC15_LDAC_N: now also U96.15 (OUTA)
- net DAC15_SCLK: now also U96.13 (OUTC)
- net DAC15_SDIN: now also U96.14 (OUTB)
- net DAC15_SDO: now also U96.10 (INF)
- net DAC15_SYNC_N: now also U96.12 (OUTD)
- net DAC16_LDAC_N: now also U97.15 (OUTA)
- net DAC16_SCLK: now also U97.13 (OUTC)
- net DAC16_SDIN: now also U97.14 (OUTB)
- net DAC16_SDO: now also U97.10 (INF)
- net DAC16_SYNC_N: now also U97.12 (OUTD)
- net DAC17_LDAC_N: now also U98.15 (OUTA)
- net DAC17_SCLK: now also U98.13 (OUTC)
- net DAC17_SDIN: now also U98.14 (OUTB)
- net DAC17_SDO: now also U98.10 (INF)
- net DAC17_SYNC_N: now also U98.12 (OUTD)
- net DAC18_LDAC_N: now also U99.15 (OUTA)
- net DAC18_SCLK: now also U99.13 (OUTC)
- net DAC18_SDIN: now also U99.14 (OUTB)
- net DAC18_SDO: now also U99.10 (INF)
- net DAC18_SYNC_N: now also U99.12 (OUTD)
- net DGND: now also U94.9 (GND2), U95.9 (GND2), U96.9 (GND2), U97.9 (GND2), U98.9 (GND2), U99.9 (GND2)
- net LDAC_N_CH13: now also U94.2 (INA)
- net LDAC_N_CH14: now also U95.2 (INA)
- net LDAC_N_CH15: now also U96.2 (INA)
- net LDAC_N_CH16: now also U97.2 (INA)
- net LDAC_N_CH17: now also U98.2 (INA)
- net LDAC_N_CH18: now also U99.2 (INA)
- net MISO_CH13: now also U94.7 (OUTF)
- net MISO_CH14: now also U95.7 (OUTF)
- net MISO_CH15: now also U96.7 (OUTF)
- net MISO_CH16: now also U97.7 (OUTF)
- net MISO_CH17: now also U98.7 (OUTF)
- net MISO_CH18: now also U99.7 (OUTF)
- net MOSI_CH13: now also U94.3 (INB)
- net MOSI_CH14: now also U95.3 (INB)
- net MOSI_CH15: now also U96.3 (INB)
- net MOSI_CH16: now also U97.3 (INB)
- net MOSI_CH17: now also U98.3 (INB)
- net MOSI_CH18: now also U99.3 (INB)
- net NGND: now also U94.8 (GND1), U95.8 (GND1), U96.8 (GND1), U97.8 (GND1), U98.8 (GND1), U99.8 (GND1)
- net SCLK_CH13: now also U94.4 (INC)
- net SCLK_CH14: now also U95.4 (INC)
- net SCLK_CH15: now also U96.4 (INC)
- net SCLK_CH16: now also U97.4 (INC)
- net SCLK_CH17: now also U98.4 (INC)
- net SCLK_CH18: now also U99.4 (INC)
- net +3V3N renamed VCCN
- net VCCN: now also U94.1 (VCC1), U95.1 (VCC1), U96.1 (VCC1), U97.1 (VCC1), U98.1 (VCC1), U99.1 (VCC1)

Commit message: adding more capacitors to analog side
Parts:
- U94, U95, U96, U97, U98, U99: footprint ISO6761:SOIC16_DW_TEX -> Package_SO:SOIC-16W_7.5x10.3mm_P1.27mm
Changed lines of the file:
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@@
 			)
 		)
-		(property "Footprint" "ISO6761:SOIC16_DW_TEX"
+		(property "Footprint" "Package_SO:SOIC-16W_7.5x10.3mm_P1.27mm"
 			(at 77.47 125.73 0)
 			(effects
@@
 			)
 		)
-		(property "Footprint" "ISO6761:SOIC16_DW_TEX"
+		(property "Footprint" "Package_SO:SOIC-16W_7.5x10.3mm_P1.27mm"
 			(at 176.53 83.82 0)
 			(effects
@@
 			)
 		)
-		(property "Footprint" "ISO6761:SOIC16_DW_TEX"
+		(property "Footprint" "Package_SO:SOIC-16W_7.5x10.3mm_P1.27mm"
 			(at 176.53 125.73 0)
 			(effects
@@
 			)
 		)
-		(property "Footprint" "ISO6761:SOIC16_DW_TEX"
+		(property "Footprint" "Package_SO:SOIC-16W_7.5x10.3mm_P1.27mm"
 			(at 77.47 43.18 0)
 			(effects
@@
 			)
 		)
-		(property "Footprint" "ISO6761:SOIC16_DW_TEX"
+		(property "Footprint" "Package_SO:SOIC-16W_7.5x10.3mm_P1.27mm"
 			(at 77.47 83.82 0)
 			(effects
@@
 			)
 		)
-		(property "Footprint" "ISO6761:SOIC16_DW_TEX"
+		(property "Footprint" "Package_SO:SOIC-16W_7.5x10.3mm_P1.27mm"
 			(at 176.53 43.18 0)
 			(effects
