File: src/pcb/dacboard/isolator1-6.kicad_sch (KiCad schematic)
At the start: 18 parts, among them U83 ISO7761FQDBQRQ1, U84 ISO7761FQDBQRQ1, U85 ISO7761FQDBQRQ1, U86 ISO7761FQDBQRQ1, U87 ISO7761FQDBQRQ1, U88 ISO7761FQDBQRQ1

Commit message: dacboard routing
Parts:
- removed U83, U84, U85, U86, U87, U88: ISO7761FQDBQRQ1, DBQ16_TEX, symbol 2025-11-18_20-36-36:ISO7761FQDBQRQ1
- added U58, U83, U84, U85, U86, U87: ISO6761FQDWRQ1, ISO6761:SOIC16_DW_TEX, symbol 2025-11-20_00-47-15:ISO6761FQDWRQ1
- C72, C73, C74, C75, C76, C77, C78, C79, C80, C81, C82, C83: footprint (none) -> Capacitor_SMD:C_0402_1005Metric_Pad0.74x0.62mm_HandSolder
Connections:
- net +5VD: now also U58.16 (VCC2), U83.16 (VCC2), U84.16 (VCC2), U85.16 (VCC2), U86.16 (VCC2), U87.16 (VCC2)
- net CLR_N: now also U83.11 (OUTE)
- net CLR_N_ALLCH: now also U83.6 (INE)
- net CS_N_CH1: now also U58.5 (IND)
- net CS_N_CH2: now also U83.5 (IND)
- net CS_N_CH3: now also U84.5 (IND)
- net CS_N_CH4: now also U85.5 (IND)
- net CS_N_CH5: now also U86.5 (IND)
- net CS_N_CH6: now also U87.5 (IND)
- net DAC1_LDAC_N: now also U58.15 (OUTA)
- net DAC1_SCLK: now also U58.13 (OUTC)
- net DAC1_SDIN: now also U58.14 (OUTB)
- net DAC1_SDO: now also U58.10 (INF)
- net DAC1_SYNC_N: now also U58.12 (OUTD)
- net DAC2_LDAC_N: now also U83.15 (OUTA)
- net DAC2_SCLK: now also U83.13 (OUTC)
- net DAC2_SDIN: now also U83.14 (OUTB)
- net DAC2_SDO: now also U83.10 (INF)
- net DAC2_SYNC_N: now also U83.12 (OUTD)
- net DAC3_LDAC_N: now also U84.15 (OUTA)
- net DAC3_SCLK: now also U84.13 (OUTC)
- net DAC3_SDIN: now also U84.14 (OUTB)
- net DAC3_SDO: now also U84.10 (INF)
- net DAC3_SYNC_N: now also U84.12 (OUTD)
- net DAC4_LDAC_N: now also U85.15 (OUTA)
- net DAC4_SCLK: now also U85.13 (OUTC)
- net DAC4_SDIN: now also U85.14 (OUTB)
- net DAC4_SDO: now also U85.10 (INF)
- net DAC4_SYNC_N: now also U85.12 (OUTD)
- net DAC5_LDAC_N: now also U86.15 (OUTA)
- net DAC5_SCLK: now also U86.13 (OUTC)
- net DAC5_SDIN: now also U86.14 (OUTB)
- net DAC5_SDO: now also U86.10 (INF)
- net DAC5_SYNC_N: now also U86.12 (OUTD)
- net DAC6_LDAC_N: now also U87.15 (OUTA)
- net DAC6_SCLK: now also U87.13 (OUTC)
- net DAC6_SDIN: now also U87.14 (OUTB)
- net DAC6_SDO: now also U87.10 (INF)
- net DAC6_SYNC_N: now also U87.12 (OUTD)
- net DGND: now also U58.9 (GND2), U83.9 (GND2), U84.9 (GND2), U85.9 (GND2), U86.9 (GND2), U87.9 (GND2)
- net LDAC_N_CH1: now also U58.2 (INA)
- net LDAC_N_CH2: now also U83.2 (INA)
- net LDAC_N_CH3: now also U84.2 (INA)
- net LDAC_N_CH4: now also U85.2 (INA)
- net LDAC_N_CH5: now also U86.2 (INA)
- net LDAC_N_CH6: now also U87.2 (INA)
- net MISO_CH1: now also U58.7 (OUTF)
- net MISO_CH2: now also U83.7 (OUTF)
- net MISO_CH3: now also U84.7 (OUTF)
- net MISO_CH4: now also U85.7 (OUTF)
- net MISO_CH5: now also U86.7 (OUTF)
- net MISO_CH6: now also U87.7 (OUTF)
- net MOSI_CH1: now also U58.3 (INB)
- net MOSI_CH2: now also U83.3 (INB)
- net MOSI_CH3: now also U84.3 (INB)
- net MOSI_CH4: now also U85.3 (INB)
- net MOSI_CH5: now also U86.3 (INB)
- net MOSI_CH6: now also U87.3 (INB)
- net NGND: now also U58.8 (GND1), U83.8 (GND1), U84.8 (GND1), U85.8 (GND1), U86.8 (GND1), U87.8 (GND1)
- net RESET_N: now also U58.11 (OUTE)
- net RESET_N_ALLCH: now also U58.6 (INE)
- net SCLK_CH1: now also U58.4 (INC)
- net SCLK_CH2: now also U83.4 (INC)
- net SCLK_CH3: now also U84.4 (INC)
- net SCLK_CH4: now also U85.4 (INC)
- net SCLK_CH5: now also U86.4 (INC)
- net SCLK_CH6: now also U87.4 (INC)
- net +3V3N renamed VCCN
- net VCCN: now also U58.1 (VCC1), U83.1 (VCC1), U84.1 (VCC1), U85.1 (VCC1), U86.1 (VCC1), U87.1 (VCC1)

Commit message: low noise digital finished
Connections:
- net CLR_N: now also U87.11 (OUTE); no longer U83.11 (OUTE)
- net CLR_N_ALLCH: now also U87.6 (INE); no longer U83.6 (INE)
- net RESET_N: no longer names the net of U58.11 (OUTE)
- net RESET_N_ALLCH: no longer names the net of U58.6 (INE)
- no-connect marks 8 -> 10

Commit message: adding more capacitors to analog side
Parts:
- U58: footprint ISO6761:SOIC16_DW_TEX -> Package_SO:SOIC-16W_7.5x12.8mm_P1.27mm
- U83, U84, U85, U86, U87: footprint ISO6761:SOIC16_DW_TEX -> Package_SO:SOIC-16W_7.5x10.3mm_P1.27mm
Changed lines of the file:
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@@
 			)
 		)
-		(property "Footprint" "ISO6761:SOIC16_DW_TEX"
+		(property "Footprint" "Package_SO:SOIC-16W_7.5x10.3mm_P1.27mm"
 			(at 72.39 81.28 0)
 			(effects
@@
 			)
 		)
-		(property "Footprint" "ISO6761:SOIC16_DW_TEX"
+		(property "Footprint" "Package_SO:SOIC-16W_7.5x10.3mm_P1.27mm"
 			(at 171.45 81.28 0)
 			(effects
@@
 			)
 		)
-		(property "Footprint" "ISO6761:SOIC16_DW_TEX"
+		(property "Footprint" "Package_SO:SOIC-16W_7.5x10.3mm_P1.27mm"
 			(at 72.39 123.19 0)
 			(effects
@@
 			)
 		)
-		(property "Footprint" "ISO6761:SOIC16_DW_TEX"
+		(property "Footprint" "Package_SO:SOIC-16W_7.5x12.8mm_P1.27mm"
 			(at 72.39 40.64 0)
 			(effects
@@
 			)
 		)
-		(property "Footprint" "ISO6761:SOIC16_DW_TEX"
+		(property "Footprint" "Package_SO:SOIC-16W_7.5x10.3mm_P1.27mm"
 			(at 171.45 123.19 0)
 			(effects
@@
 			)
 		)
-		(property "Footprint" "ISO6761:SOIC16_DW_TEX"
+		(property "Footprint" "Package_SO:SOIC-16W_7.5x10.3mm_P1.27mm"
 			(at 171.45 40.64 0)
 			(effects

Commit message: got rid of all drc errors
Parts:
- U58: footprint Package_SO:SOIC-16W_7.5x12.8mm_P1.27mm -> Package_SO:SOIC-16W_7.5x10.3mm_P1.27mm
Changed lines of the file:
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@@
 			)
 		)
-		(property "Footprint" "Package_SO:SOIC-16W_7.5x12.8mm_P1.27mm"
+		(property "Footprint" "Package_SO:SOIC-16W_7.5x10.3mm_P1.27mm"
 			(at 72.39 40.64 0)
 			(effects
