File: pcb/dacboard-new/dac19-24.kicad_sch (KiCad schematic)
At the start: 30 parts, among them U46 AD8676xR, U47 AD8676xR, U48 AD8676xR, U49 AD8676xR, U50 AD5791BRUZ, U51 AD5791BRUZ, U52 AD5791BRUZ, U53 AD5791BRUZ, U54 AD8676xR, U55 AD8676xR, U56 AD5791BRUZ, U57 AD5791BRUZ

Commit message: new pcb progress
Parts:
- added R78, R79, R80, R81, R82, R83, R84, R85, R86, R87, R88, R89: 10K, Resistor_SMD:R_0402_1005Metric_Pad0.72x0.64mm_HandSolder, symbol Device:R_US
Connections:
- net +5VD: now also R78.1, R79.1, R80.1, R81.1, R82.1, R83.1, R84.1, R85.1, R86.1, R87.1, R88.1, R89.1
- removed net CLR_N: U50.7 (*CLR), U51.7 (*CLR), U52.7 (*CLR), U53.7 (*CLR), U56.7 (*CLR), U57.7 (*CLR)
- removed net RESET_N: U50.6 (*RESET), U51.6 (*RESET), U52.6 (*RESET), U53.6 (*RESET), U56.6 (*RESET), U57.6 (*RESET)
- new net: R79.2, U50.7 (*CLR)
- new net: R78.2, U50.6 (*RESET)
- new net: R84.2, U53.6 (*RESET)
- new net: R81.2, U51.7 (*CLR)
- new net: R87.2, U56.7 (*CLR)
- new net: R89.2, U57.7 (*CLR)
- new net: R86.2, U56.6 (*RESET)
- new net: R85.2, U53.7 (*CLR)
- new net: R88.2, U57.6 (*RESET)
- new net: R82.2, U52.6 (*RESET)
- new net: R83.2, U52.7 (*CLR)
- new net: R80.2, U51.6 (*RESET)
