File: pcb/dacboard-new/dacboard.kicad_pcb (KiCad board)
At the start: 14 copper layers, 374 parts, among them J1 Screw_Terminal_01x03, J2 Screw_Terminal_01x02, J23 Conn_01x05, J24 Conn_01x03, J25 Conn_01x02, J26 Screw_Terminal_01x02, J27 ASP-184330-01, J28 Conn_02x12_Odd_Even, J29 Conn_02x12_Odd_Even, J3 Conn_01x30_Socket, J30 Conn_02x12_Odd_Even, J31 Conn_02x12_Odd_Even, U1 LTC6655CHMS8-2.5_PBF, U10 AD5791BRUZ, U100 ISO6761FQDWRQ1, U101 ISO6761FQDWRQ1, U102 ISO6761FQDWRQ1, U103 ISO6761FQDWRQ1, U104 ISO6761FQDWRQ1, U105 ISO6761FQDWRQ1, U11 AD8676xR, U12 AD8676xR, U13 AD5791BRUZ, U14 AD8676xR, U15 AD5791BRUZ, U16 AD8676xR, U17 AD5791BRUZ, U18 AD8676xR, U19 AD5791BRUZ, U2 LTC6655CHMS8-2.5_PBF, U20 AD8676xR, U21 AD5791BRUZ, U22 AD8676xR, U23 AD8676xR, U24 AD8676xR, U25 AD8676xR, U26 AD5791BRUZ, U27 AD5791BRUZ, U28 AD5791BRUZ, U29 AD5791BRUZ, U3 LTC6655CHMS8-2.5_PBF, U30 AD8676xR, U31 AD8676xR, U32 AD5791BRUZ, U33 AD5791BRUZ, U34 AD8676xR, U35 AD8676xR, U36 AD8676xR, U37 AD8676xR, U38 AD5791BRUZ, U39 AD5791BRUZ, U4 LTC6655CHMS8-2.5_PBF, U40 AD5791BRUZ, U41 AD5791BRUZ, U42 AD8676xR, U43 AD8676xR, U44 AD5791BRUZ, U45 AD5791BRUZ, U46 AD8676xR, U47 AD8676xR, U48 AD8676xR, U49 AD8676xR, U5 LTC6655CHMS8-2.5_PBF, U50 AD5791BRUZ, U51 AD5791BRUZ, U52 AD5791BRUZ, U53 AD5791BRUZ, U54 AD8676xR, U55 AD8676xR, U56 AD5791BRUZ, U57 AD5791BRUZ, U58 ISO6761FQDWRQ1, U59 AD8675ARZ, U6 LTC6655CHMS8-2.5_PBF, U60 AD8675ARZ, U61 AD8675ARZ, U62 AD8675ARZ, U63 AD8675ARZ, U64 AD8675ARZ, U65 AD8675ARZ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

Commit message: new pcb progress
Parts:
- removed R41: R_US, Resistor_THT:R_Axial_DIN0309_L9.0mm_D3.2mm_P20.32mm_Horizontal
- added J10: RFPC-SMA28-F, RFPC-SMA28-F:GRADCONN_RFPC-SMA28-F, F.Cu at (271.9, 94.3)
- added J11: RFPC-SMA28-F, RFPC-SMA28-F:GRADCONN_RFPC-SMA28-F, F.Cu at (281.9, 119.3)
- added J12: RFPC-SMA28-F, RFPC-SMA28-F:GRADCONN_RFPC-SMA28-F, F.Cu at (251.9, 94.3)
- added J13: RFPC-SMA28-F, RFPC-SMA28-F:GRADCONN_RFPC-SMA28-F, F.Cu at (261.9, 119.3)
- added J14: RFPC-SMA28-F, RFPC-SMA28-F:GRADCONN_RFPC-SMA28-F, F.Cu at (231.9, 94.3)
- added J15: RFPC-SMA28-F, RFPC-SMA28-F:GRADCONN_RFPC-SMA28-F, F.Cu at (241.9, 119.3)
- added J16: RFPC-SMA28-F, RFPC-SMA28-F:GRADCONN_RFPC-SMA28-F, F.Cu at (157.9, 119.3)
- added J17: RFPC-SMA28-F, RFPC-SMA28-F:GRADCONN_RFPC-SMA28-F, F.Cu at (167.9, 94.3)
- added J18: RFPC-SMA28-F, RFPC-SMA28-F:GRADCONN_RFPC-SMA28-F, F.Cu at (137.9, 119.3)
- added J19: RFPC-SMA28-F, RFPC-SMA28-F:GRADCONN_RFPC-SMA28-F, F.Cu at (147.9, 94.3)
- added J20: RFPC-SMA28-F, RFPC-SMA28-F:GRADCONN_RFPC-SMA28-F, F.Cu at (117.9, 119.3)
- added J21: RFPC-SMA28-F, RFPC-SMA28-F:GRADCONN_RFPC-SMA28-F, F.Cu at (127.9, 94.3)
- added J22: RFPC-SMA28-F, RFPC-SMA28-F:GRADCONN_RFPC-SMA28-F, F.Cu at (97.9, 119.3)
- added J32: RFPC-SMA28-F, RFPC-SMA28-F:GRADCONN_RFPC-SMA28-F, F.Cu at (107.9, 94.3)
- added J33: RFPC-SMA28-F, RFPC-SMA28-F:GRADCONN_RFPC-SMA28-F, F.Cu at (77.9, 119.3)
- added J34: RFPC-SMA28-F, RFPC-SMA28-F:GRADCONN_RFPC-SMA28-F, F.Cu at (87.9, 94.3)
- added J35: RFPC-SMA28-F, RFPC-SMA28-F:GRADCONN_RFPC-SMA28-F, F.Cu at (57.9, 119.3)
- added J36: RFPC-SMA28-F, RFPC-SMA28-F:GRADCONN_RFPC-SMA28-F, F.Cu at (67.9, 94.3)
- added J37: Screw_Terminal_01x03, TerminalBlock_Phoenix:TerminalBlock_Phoenix_MKDS-1,5-3-5.08_1x03_P5.08mm_Horizontal, F.Cu at (216.0, 164.4)
- added J38: Screw_Terminal_01x02, TerminalBlock_Phoenix:TerminalBlock_Phoenix_MKDS-1,5-2-5.08_1x02_P5.08mm_Horizontal, F.Cu at (182.7, 184.6)
- added J39: Screw_Terminal_01x02, TerminalBlock_Phoenix:TerminalBlock_Phoenix_MKDS-1,5-2-5.08_1x02_P5.08mm_Horizontal, F.Cu at (217.2, 189.6)
- added J4: RFPC-SMA28-F, RFPC-SMA28-F:GRADCONN_RFPC-SMA28-F, F.Cu at (331.9, 94.3)
- added J40: Conn_01x05, Connector_PinHeader_2.54mm:PinHeader_1x05_P2.54mm_Vertical, F.Cu at (174.8, 119.2)
- added J41: Conn_01x05, Connector_PinHeader_2.54mm:PinHeader_1x05_P2.54mm_Vertical, F.Cu at (224.2, 119.2)
- added J42: Conn_01x03, Connector_PinHeader_2.54mm:PinHeader_1x03_P2.54mm_Vertical, F.Cu at (213.7, 175.8)
- added J43: Conn_01x03, Connector_PinHeader_2.54mm:PinHeader_1x03_P2.54mm_Vertical, F.Cu at (180.3, 175.5)
- added J44: Conn_01x02, Connector_PinHeader_2.54mm:PinHeader_1x02_P2.54mm_Vertical, F.Cu at (230.3, 212.2)
- added J45: Conn_01x02, Connector_PinHeader_2.54mm:PinHeader_1x02_P2.54mm_Vertical, F.Cu at (234.9, 212.2)
- added J46: Conn_01x05, Connector_PinHeader_2.54mm:PinHeader_1x05_P2.54mm_Vertical, F.Cu at (334.8, 69.3)
- added J47: Conn_01x03, Connector_PinHeader_2.54mm:PinHeader_1x03_P2.54mm_Vertical, F.Cu at (54.2, 182.6)
- added J48: Conn_01x02, Connector_PinHeader_2.54mm:PinHeader_1x02_P2.54mm_Vertical, F.Cu at (239.5, 212.2)
- added J5: RFPC-SMA28-F, RFPC-SMA28-F:GRADCONN_RFPC-SMA28-F, F.Cu at (341.9, 119.3)
- added J6: RFPC-SMA28-F, RFPC-SMA28-F:GRADCONN_RFPC-SMA28-F, F.Cu at (311.9, 94.3)
- added J7: RFPC-SMA28-F, RFPC-SMA28-F:GRADCONN_RFPC-SMA28-F, F.Cu at (321.9, 119.3)
- added J8: RFPC-SMA28-F, RFPC-SMA28-F:GRADCONN_RFPC-SMA28-F, F.Cu at (291.9, 94.3)
- added J9: RFPC-SMA28-F, RFPC-SMA28-F:GRADCONN_RFPC-SMA28-F, F.Cu at (301.9, 119.3)
- added R42: 10K, Resistor_SMD:R_0402_1005Metric_Pad0.72x0.64mm_HandSolder, F.Cu at (247.7, 170.6)
- added R42: 10K, Resistor_SMD:R_0402_1005Metric_Pad0.72x0.64mm_HandSolder, F.Cu at (57.6, 170.6)
- added R42: 10K, Resistor_SMD:R_0402_1005Metric_Pad0.72x0.64mm_HandSolder, F.Cu at (137.7, 170.6)
- added R42: 10K, Resistor_SMD:R_0402_1005Metric_Pad0.72x0.64mm_HandSolder, F.Cu at (77.7, 170.6)
- added R42: 10K, Resistor_SMD:R_0402_1005Metric_Pad0.72x0.64mm_HandSolder, B.Cu at (72.1, 170.6)
- added R42: 10K, Resistor_SMD:R_0402_1005Metric_Pad0.72x0.64mm_HandSolder, B.Cu at (262.1, 170.6)
- added R42: 10K, Resistor_SMD:R_0402_1005Metric_Pad0.72x0.64mm_HandSolder, B.Cu at (112.1, 170.6)
- added R42: 10K, Resistor_SMD:R_0402_1005Metric_Pad0.72x0.64mm_HandSolder, B.Cu at (152.1, 170.6)
- added R42: 10K, Resistor_SMD:R_0402_1005Metric_Pad0.72x0.64mm_HandSolder, B.Cu at (322.1, 170.6)
- added R42: 10K, Resistor_SMD:R_0402_1005Metric_Pad0.72x0.64mm_HandSolder, B.Cu at (92.1, 170.6)
- added R42: 10K, Resistor_SMD:R_0402_1005Metric_Pad0.72x0.64mm_HandSolder, B.Cu at (282.1, 170.6)
- added R42: 10K, Resistor_SMD:R_0402_1005Metric_Pad0.72x0.64mm_HandSolder, F.Cu at (97.7, 170.6)
- added R42: 10K, Resistor_SMD:R_0402_1005Metric_Pad0.72x0.64mm_HandSolder, B.Cu at (132.1, 170.6)
- added R42: 10K, Resistor_SMD:R_0402_1005Metric_Pad0.72x0.64mm_HandSolder, B.Cu at (302.1, 170.6)
- added R42: 10K, Resistor_SMD:R_0402_1005Metric_Pad0.72x0.64mm_HandSolder, B.Cu at (242.1, 170.6)
- added R42: 10K, Resistor_SMD:R_0402_1005Metric_Pad0.72x0.64mm_HandSolder, B.Cu at (172.1, 170.6)
- added R42: 10K, Resistor_SMD:R_0402_1005Metric_Pad0.72x0.64mm_HandSolder, B.Cu at (342.1, 170.6)
- added R42: 10K, Resistor_SMD:R_0402_1005Metric_Pad0.72x0.64mm_HandSolder, F.Cu at (307.6, 170.6)
- added R42: 10K, Resistor_SMD:R_0402_1005Metric_Pad0.72x0.64mm_HandSolder, F.Cu at (267.6, 170.6)
- added R42: 10K, Resistor_SMD:R_0402_1005Metric_Pad0.72x0.64mm_HandSolder, F.Cu at (227.7, 170.6)
- added R42: 10K, Resistor_SMD:R_0402_1005Metric_Pad0.72x0.64mm_HandSolder, F.Cu at (287.6, 170.6)
- added R42: 10K, Resistor_SMD:R_0402_1005Metric_Pad0.72x0.64mm_HandSolder, F.Cu at (117.7, 170.6)
- added R42: 10K, Resistor_SMD:R_0402_1005Metric_Pad0.72x0.64mm_HandSolder, F.Cu at (327.6, 170.6)
- added R42: 10K, Resistor_SMD:R_0402_1005Metric_Pad0.72x0.64mm_HandSolder, F.Cu at (157.7, 170.6)
- added R44: 10K, Resistor_SMD:R_0402_1005Metric_Pad0.72x0.64mm_HandSolder, F.Cu at (268.1, 172.2)
- added R44: 10K, Resistor_SMD:R_0402_1005Metric_Pad0.72x0.64mm_HandSolder, F.Cu at (58.0, 172.2)
- added R44: 10K, Resistor_SMD:R_0402_1005Metric_Pad0.72x0.64mm_HandSolder, F.Cu at (228.1, 172.2)
- added R44: 10K, Resistor_SMD:R_0402_1005Metric_Pad0.72x0.64mm_HandSolder, F.Cu at (138.1, 172.2)
- added R44: 10K, Resistor_SMD:R_0402_1005Metric_Pad0.72x0.64mm_HandSolder, B.Cu at (301.7, 172.2)
- added R44: 10K, Resistor_SMD:R_0402_1005Metric_Pad0.72x0.64mm_HandSolder, B.Cu at (111.7, 172.2)
- added R44: 10K, Resistor_SMD:R_0402_1005Metric_Pad0.72x0.64mm_HandSolder, B.Cu at (171.7, 172.2)
- added R44: 10K, Resistor_SMD:R_0402_1005Metric_Pad0.72x0.64mm_HandSolder, B.Cu at (241.7, 172.2)
- added R44: 10K, Resistor_SMD:R_0402_1005Metric_Pad0.72x0.64mm_HandSolder, B.Cu at (151.7, 172.2)
- added R44: 10K, Resistor_SMD:R_0402_1005Metric_Pad0.72x0.64mm_HandSolder, B.Cu at (341.7, 172.2)
- added R44: 10K, Resistor_SMD:R_0402_1005Metric_Pad0.72x0.64mm_HandSolder, B.Cu at (91.7, 172.2)
- added R44: 10K, Resistor_SMD:R_0402_1005Metric_Pad0.72x0.64mm_HandSolder, F.Cu at (158.1, 172.2)
- added R44: 10K, Resistor_SMD:R_0402_1005Metric_Pad0.72x0.64mm_HandSolder, B.Cu at (261.7, 172.2)
- added R44: 10K, Resistor_SMD:R_0402_1005Metric_Pad0.72x0.64mm_HandSolder, B.Cu at (71.7, 172.2)
- added R44: 10K, Resistor_SMD:R_0402_1005Metric_Pad0.72x0.64mm_HandSolder, B.Cu at (321.7, 172.2)
- added R44: 10K, Resistor_SMD:R_0402_1005Metric_Pad0.72x0.64mm_HandSolder, B.Cu at (131.7, 172.2)
- added R44: 10K, Resistor_SMD:R_0402_1005Metric_Pad0.72x0.64mm_HandSolder, B.Cu at (281.7, 172.2)
- added R44: 10K, Resistor_SMD:R_0402_1005Metric_Pad0.72x0.64mm_HandSolder, F.Cu at (98.0, 172.2)
- added R44: 10K, Resistor_SMD:R_0402_1005Metric_Pad0.72x0.64mm_HandSolder, F.Cu at (78.0, 172.2)
- added R44: 10K, Resistor_SMD:R_0402_1005Metric_Pad0.72x0.64mm_HandSolder, F.Cu at (308.1, 172.2)
- added R44: 10K, Resistor_SMD:R_0402_1005Metric_Pad0.72x0.64mm_HandSolder, F.Cu at (248.1, 172.2)
- added R44: 10K, Resistor_SMD:R_0402_1005Metric_Pad0.72x0.64mm_HandSolder, F.Cu at (288.1, 172.2)
- added R44: 10K, Resistor_SMD:R_0402_1005Metric_Pad0.72x0.64mm_HandSolder, F.Cu at (118.0, 172.2)
- added R44: 10K, Resistor_SMD:R_0402_1005Metric_Pad0.72x0.64mm_HandSolder, F.Cu at (328.1, 172.2)
- J2: footprint TerminalBlock_4Ucon:TerminalBlock_4Ucon_1x02_P3.50mm_Horizontal -> TerminalBlock_Phoenix:TerminalBlock_Phoenix_MKDS-1,5-2-5.08_1x02_P5.08mm_Horizontal
- J26: value Screw_Terminal_01x02 -> Screw_Terminal_01x03; footprint TerminalBlock_4Ucon:TerminalBlock_4Ucon_1x02_P3.50mm_Horizontal -> TerminalBlock_Phoenix:TerminalBlock_Phoenix_MKDS-1,5-3-5.08_1x03_P5.08mm_Horizontal
- J27: moved to B.Cu
- J3: value Conn_01x30_Socket -> DLS3XS6AK44X; footprint Connector_PinHeader_2.54mm:PinHeader_1x30_P2.54mm_Horizontal -> DLS3XS6AK44X:CONN_DLS3XS6AK44X_CEC; moved to F.Cu
- moved J1 141.5 mm to (194.8, 162.4)
- moved J26 132.7 mm to (183.6, 154.3), turned to -90 degrees
- moved J23 97.3 mm to (65.9, 66.3), turned to -45 degrees
- moved J2 85.1 mm to (197.7, 187.7)
- moved REF** 80.1 mm to (343.0, 66.1)
- moved C124 60.0 mm to (59.9, 161.3)
- moved C125 60.0 mm to (79.9, 161.3)
- moved C126 60.0 mm to (99.9, 161.3)
- moved C127 60.0 mm to (119.9, 161.3)
- moved C128 60.0 mm to (139.9, 161.3)
- moved C129 60.0 mm to (159.9, 161.3)
- moved C131 60.0 mm to (229.9, 161.3)
- moved C133 60.0 mm to (249.9, 161.3)
- moved C135 60.0 mm to (269.9, 161.3)
- moved C137 60.0 mm to (289.9, 161.3)
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Connections:
- J26 pad 1: VCCN -> VDD
- J26 pad 2: NGND -> AGND
- J3 pad 1: AGND -> BUF1_VOUT
- J3 pad 10: BUF11_VOUT -> BUF10_VOUT
- J3 pad 11: BUF22_VOUT -> BUF11_VOUT
- J3 pad 12: BUF10_VOUT -> BUF12_VOUT
- J3 pad 13: BUF21_VOUT -> BUF13_VOUT
- J3 pad 14: BUF9_VOUT -> BUF14_VOUT
- J3 pad 15: BUF20_VOUT -> BUF15_VOUT
- J3 pad 16: BUF8_VOUT -> BUF16_VOUT
- J3 pad 17: BUF19_VOUT -> BUF17_VOUT
- J3 pad 18: BUF7_VOUT -> BUF18_VOUT
- J3 pad 19: BUF18_VOUT -> BUF19_VOUT
- J3 pad 2: AGND -> BUF2_VOUT
- J3 pad 20: BUF6_VOUT -> BUF20_VOUT
- J3 pad 21: BUF17_VOUT -> BUF21_VOUT
- J3 pad 22: BUF5_VOUT -> BUF22_VOUT
- J3 pad 23: BUF16_VOUT -> BUF23_VOUT
- J3 pad 24: BUF4_VOUT -> BUF24_VOUT
- J3 pad 25: BUF15_VOUT -> unconnected-(J3-Pad25)
- J3 pad 26: BUF3_VOUT -> (no net)
- J3 pad 27: BUF14_VOUT -> (no net)
- J3 pad 3: AGND -> BUF3_VOUT
- J3 pad 4: AGND -> BUF4_VOUT
- J3 pad 5: AGND -> BUF5_VOUT
- J3 pad 6: AGND -> BUF6_VOUT
- J3 pad 7: BUF24_VOUT -> BUF7_VOUT
- J3 pad 8: BUF12_VOUT -> BUF8_VOUT
- J3 pad 9: BUF23_VOUT -> BUF9_VOUT
- U10 pad 6: RESET_N -> Net-(U10-*RESET)
- U10 pad 7: CLR_N -> Net-(U10-*CLR)
- U13 pad 6: RESET_N -> Net-(U13-*RESET)
- U13 pad 7: CLR_N -> Net-(U13-*CLR)
- U15 pad 6: RESET_N -> Net-(U15-*RESET)
- U15 pad 7: CLR_N -> Net-(U15-*CLR)
- U17 pad 6: RESET_N -> Net-(U17-*RESET)
- U17 pad 7: CLR_N -> Net-(U17-*CLR)
- U19 pad 6: RESET_N -> Net-(U19-*RESET)
- U19 pad 7: CLR_N -> Net-(U19-*CLR)
- U21 pad 6: RESET_N -> Net-(U21-*RESET)
- U21 pad 7: CLR_N -> Net-(U21-*CLR)
- U26 pad 6: RESET_N -> Net-(U26-*RESET)
- U26 pad 7: CLR_N -> Net-(U26-*CLR)
- U27 pad 6: RESET_N -> Net-(U27-*RESET)
- U27 pad 7: CLR_N -> Net-(U27-*CLR)
- U28 pad 6: RESET_N -> Net-(U28-*RESET)
- U28 pad 7: CLR_N -> Net-(U28-*CLR)
- U29 pad 6: RESET_N -> Net-(U29-*RESET)
- U29 pad 7: CLR_N -> Net-(U29-*CLR)
- U32 pad 6: RESET_N -> Net-(U32-*RESET)
- U32 pad 7: CLR_N -> Net-(U32-*CLR)
- U33 pad 6: RESET_N -> Net-(U33-*RESET)
- U33 pad 7: CLR_N -> Net-(U33-*CLR)
- U38 pad 6: RESET_N -> Net-(U38-*RESET)
- U38 pad 7: CLR_N -> Net-(U38-*CLR)
- U39 pad 6: RESET_N -> Net-(U39-*RESET)
- U39 pad 7: CLR_N -> Net-(U39-*CLR)
- U40 pad 6: RESET_N -> Net-(U40-*RESET)
- U40 pad 7: CLR_N -> Net-(U40-*CLR)
- U41 pad 6: RESET_N -> Net-(U41-*RESET)
- U41 pad 7: CLR_N -> Net-(U41-*CLR)
- U44 pad 6: RESET_N -> Net-(U44-*RESET)
- U44 pad 7: CLR_N -> Net-(U44-*CLR)
- U45 pad 6: RESET_N -> Net-(U45-*RESET)
- U45 pad 7: CLR_N -> Net-(U45-*CLR)
- U50 pad 6: RESET_N -> Net-(U50-*RESET)
- U50 pad 7: CLR_N -> Net-(U50-*CLR)
- U51 pad 6: RESET_N -> Net-(U51-*RESET)
- U51 pad 7: CLR_N -> Net-(U51-*CLR)
- U52 pad 6: RESET_N -> Net-(U52-*RESET)
- U52 pad 7: CLR_N -> Net-(U52-*CLR)
- U53 pad 6: RESET_N -> Net-(U53-*RESET)
- U53 pad 7: CLR_N -> Net-(U53-*CLR)
- U56 pad 6: RESET_N -> Net-(U56-*RESET)
- U56 pad 7: CLR_N -> Net-(U56-*CLR)
- U57 pad 6: RESET_N -> Net-(U57-*RESET)
- U57 pad 7: CLR_N -> Net-(U57-*CLR)
Routing:
- net BUF13_VOUT: track 0.00 -> 231.2 mm
- net BUF12_VOUT: track 0.00 -> 192.2 mm, vias 0 -> 4
- net BUF24_VOUT: track 0.00 -> 185.7 mm
- net BUF1_VOUT: track 0.00 -> 178.6 mm
- net BUF14_VOUT: track 0.00 -> 175.3 mm
- net BUF11_VOUT: track 0.00 -> 175.1 mm
- net BUF23_VOUT: track 0.00 -> 169.4 mm
- net BUF2_VOUT: track 0.00 -> 162.0 mm
- net BUF10_VOUT: track 0.00 -> 159.5 mm
- net BUF15_VOUT: track 0.00 -> 159.0 mm
- net BUF22_VOUT: track 0.00 -> 153.3 mm
- net BUF3_VOUT: track 0.00 -> 145.8 mm
- net BUF9_VOUT: track 0.00 -> 142.4 mm
- net BUF16_VOUT: track 0.00 -> 141.8 mm
- net BUF21_VOUT: track 0.00 -> 137.8 mm
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Other:
- board outline added: 296.3 x 184 mm
- copper layers 14 -> 16
