File: pcb/dacboard-new/isolator7-12.kicad_sch (KiCad schematic)
At the start: 18 parts, among them U88 ISO6761FQDWRQ1, U89 ISO6761FQDWRQ1, U90 ISO6761FQDWRQ1, U91 ISO6761FQDWRQ1, U92 ISO6761FQDWRQ1, U93 ISO6761FQDWRQ1

Commit message: finished designing new pcb
Connections:
- net MARK7_5V: now reaches U88.11 (OUTE)
- net MARK7: now reaches U88.6 (INE)
- net MARK8_5V: now reaches U89.11 (OUTE)
- net MARK8: now reaches U89.6 (INE)
- net DAC10_SDO renamed TRIG2_5V
- net DAC11_SDO renamed TRIG3_5V
- net DAC12_SDO renamed TRIG4_5V
- net DAC9_SDO renamed TRIG1_5V
- net MISO_CH10 renamed TRIG2
- net MISO_CH11 renamed TRIG3
- net MISO_CH12 renamed TRIG4
- net MISO_CH9 renamed TRIG1
- no-connect marks 12 -> 8
