File: pcb/dacboard-new/vref.kicad_sch (KiCad schematic)
At the start: 53 parts, among them J1 Screw_Terminal_01x03, J2 Screw_Terminal_01x02, J23 Conn_01x05, J24 Conn_01x03, J25 Conn_01x02, J26 Screw_Terminal_01x02, U1 LTC6655CHMS8-2.5_PBF, U2 LTC6655CHMS8-2.5_PBF, U3 LTC6655CHMS8-2.5_PBF, U4 LTC6655CHMS8-2.5_PBF, U5 LTC6655CHMS8-2.5_PBF, U6 LTC6655CHMS8-2.5_PBF, U7 LTC6655CHMS8-2.5_PBF, U8 LTC6655CHMS8-2.5_PBF, U9 AD8676xR

Commit message: new pcb progress
Parts:
- removed J26: Screw_Terminal_01x02, TerminalBlock_4Ucon:TerminalBlock_4Ucon_1x02_P3.50mm_Horizontal, symbol Connector:Screw_Terminal_01x02
- removed R41: R_US, Resistor_THT:R_Axial_DIN0309_L9.0mm_D3.2mm_P20.32mm_Horizontal, symbol Device:R_US
- added J26, J37: Screw_Terminal_01x03, TerminalBlock_Phoenix:TerminalBlock_Phoenix_MKDS-1,5-3-5.08_1x03_P5.08mm_Horizontal, symbol Connector:Screw_Terminal_01x03
- added J38, J39: Screw_Terminal_01x02, TerminalBlock_Phoenix:TerminalBlock_Phoenix_MKDS-1,5-2-5.08_1x02_P5.08mm_Horizontal, symbol Connector:Screw_Terminal_01x02
- added J40, J41, J46: Conn_01x05, Connector_PinHeader_2.54mm:PinHeader_1x05_P2.54mm_Vertical, symbol Connector_Generic:Conn_01x05
- added J42, J43, J47: Conn_01x03, Connector_PinHeader_2.54mm:PinHeader_1x03_P2.54mm_Vertical, symbol Connector_Generic:Conn_01x03
- added J44, J45, J48: Conn_01x02, Connector_PinHeader_2.54mm:PinHeader_1x02_P2.54mm_Vertical, symbol Connector_Generic:Conn_01x02
- J2: footprint TerminalBlock_4Ucon:TerminalBlock_4Ucon_1x02_P3.50mm_Horizontal -> TerminalBlock_Phoenix:TerminalBlock_Phoenix_MKDS-1,5-2-5.08_1x02_P5.08mm_Horizontal
Connections:
- net +5VD: now also J38.1 (Pin_1), J39.1 (Pin_1), J42.1 (Pin_1), J43.1 (Pin_1), J47.1 (Pin_1)
- net AGND: now also J26.2 (Pin_2), J37.2 (Pin_2), J40.2 (Pin_2), J41.2 (Pin_2), J46.2 (Pin_2)
- net DGND: now also J38.2 (Pin_2), J39.2 (Pin_2), J42.3 (Pin_3), J43.3 (Pin_3), J47.3 (Pin_3)
- net LOGIC_LEVEL: now also J42.2 (Pin_2), J43.2 (Pin_2), J47.2 (Pin_2)
- net NGND: now also J44.2 (Pin_2), J45.2 (Pin_2), J48.2 (Pin_2)
- net VCCN: now also J44.1 (Pin_1), J45.1 (Pin_1), J48.1 (Pin_1)
- net VDD: now also J26.1 (Pin_1), J37.1 (Pin_1), J40.1 (Pin_1), J41.1 (Pin_1), J46.1 (Pin_1)
- net VREF+: now also J40.4 (Pin_4), J41.4 (Pin_4), J46.4 (Pin_4)
- net VREF-: now also J40.5 (Pin_5), J41.5 (Pin_5), J46.5 (Pin_5)
- net VSS: now also J26.3 (Pin_3), J37.3 (Pin_3), J40.3 (Pin_3), J41.3 (Pin_3), J46.3 (Pin_3)
Other:
- moved on the sheet: J2

Commit message: finished designing new pcb
Parts:
- added J63: Screw_Terminal_01x02, TerminalBlock_Phoenix:TerminalBlock_Phoenix_MKDS-1,5-2-5.08_1x02_P5.08mm_Horizontal, symbol Connector:Screw_Terminal_01x02
Connections:
- net NGND: now also J63.2 (Pin_2)
- net VCCN: now also J63.1 (Pin_1)
