File: pcb/dacboard-new/dac1-6.kicad_sch (KiCad schematic)
At the start: 30 parts, among them U10 AD5791BRUZ, U11 AD8676xR, U12 AD8676xR, U13 AD5791BRUZ, U14 AD8676xR, U15 AD5791BRUZ, U16 AD8676xR, U17 AD5791BRUZ, U18 AD8676xR, U19 AD5791BRUZ, U20 AD8676xR, U21 AD5791BRUZ

Commit message: new pcb progress
Parts:
- added R42, R43, R44, R45, R46, R47, R48, R49, R50, R51, R52, R53: 10K, Resistor_SMD:R_0402_1005Metric_Pad0.72x0.64mm_HandSolder, symbol Device:R_US
Connections:
- net +5VD: now also R42.1, R43.1, R44.1, R45.1, R46.1, R47.1, R48.1, R49.1, R50.1, R51.1, R52.1, R53.1
- removed net CLR_N: U10.7 (*CLR), U13.7 (*CLR), U15.7 (*CLR), U17.7 (*CLR), U19.7 (*CLR), U21.7 (*CLR)
- removed net RESET_N: U10.6 (*RESET), U13.6 (*RESET), U15.6 (*RESET), U17.6 (*RESET), U19.6 (*RESET), U21.6 (*RESET)
- new net: R43.2, U13.6 (*RESET)
- new net: R50.2, U19.6 (*RESET)
- new net: R51.2, U19.7 (*CLR)
- new net: R46.2, U15.6 (*RESET)
- new net: R47.2, U15.7 (*CLR)
- new net: R44.2, U10.7 (*CLR)
- new net: R52.2, U21.6 (*RESET)
- new net: R53.2, U21.7 (*CLR)
- new net: R45.2, U13.7 (*CLR)
- new net: R48.2, U17.6 (*RESET)
- new net: R42.2, U10.6 (*RESET)
- new net: R49.2, U17.7 (*CLR)
