File: pcb/dacboard-new/output_header.kicad_sch (KiCad schematic)
At the start: 1 part, among them J3 Conn_01x30_Socket

Commit message: new pcb progress
Parts:
- removed J3: Conn_01x30_Socket, Connector_PinHeader_2.54mm:PinHeader_1x30_P2.54mm_Horizontal, symbol Connector:Conn_01x30_Socket
- added J10, J11, J12, J13, J14, J15, J16, J17, J18, J19, J20, J21, J22, J32, J33, J34, J35, J36, J4, J5, J6, J7, J8, J9: RFPC-SMA28-F, RFPC-SMA28-F:GRADCONN_RFPC-SMA28-F, symbol RFPC-SMA28-F:RFPC-SMA28-F
- added J3: DLS3XS6AK44X, DLS3XS6AK44X:CONN_DLS3XS6AK44X_CEC, symbol DLS3XS6AK44X:DLS3XS6AK44X
Connections:
- net AGND: now also J10.G1, J10.G2, J10.G3, J10.G4, J11.G1, J11.G2, J11.G3, J11.G4, J12.G1, J12.G2, J12.G3, J12.G4, J13.G1, J13.G2, J13.G3, J13.G4, J14.G1, J14.G2, J14.G3, J14.G4, J15.G1, J15.G2, J15.G3, J15.G4, J16.G1, J16.G2, J16.G3, J16.G4, J17.G1, J17.G2, J17.G3, J17.G4, J18.G1, J18.G2, J18.G3, J18.G4, J19.G1, J19.G2, J19.G3, J19.G4, J20.G1, J20.G2, J20.G3, J20.G4, J21.G1, J21.G2, J21.G3, J21.G4, J22.G1, J22.G2, J22.G3, J22.G4, J32.G1, J32.G2, J32.G3, J32.G4, J33.G1, J33.G2, J33.G3, J33.G4, J34.G1, J34.G2, J34.G3, J34.G4, J35.G1, J35.G2, J35.G3, J35.G4, J36.G1, J36.G2, J36.G3, J36.G4, J4.G1, J4.G2, J4.G3, J4.G4, J5.G1, J5.G2, J5.G3, J5.G4, J6.G1, J6.G2, J6.G3, J6.G4, J7.G1, J7.G2, J7.G3, J7.G4, J8.G1, J8.G2, J8.G3, J8.G4, J9.G1, J9.G2, J9.G3, J9.G4
- net BUF10_VOUT: now also J3.10, J9.1
- net BUF11_VOUT: now also J3.11, J7.1
- net BUF12_VOUT: now also J3.12, J5.1
- net BUF13_VOUT: now also J3.13, J35.1
- net BUF14_VOUT: now also J3.14, J33.1
- net BUF15_VOUT: now also J22.1, J3.15
- net BUF16_VOUT: now also J20.1, J3.16
- net BUF17_VOUT: now also J18.1, J3.17
- net BUF18_VOUT: now also J16.1, J3.18
- net BUF19_VOUT: now also J14.1, J3.19
- net BUF1_VOUT: now also J3.1, J36.1
- net BUF20_VOUT: now also J12.1, J3.20
- net BUF21_VOUT: now also J10.1, J3.21
- net BUF22_VOUT: now also J3.22, J8.1
- net BUF23_VOUT: now also J3.23, J6.1
- net BUF24_VOUT: now also J3.24, J4.1
- net BUF2_VOUT: now also J3.2, J34.1
- net BUF3_VOUT: now also J3.3, J32.1
- net BUF4_VOUT: now also J21.1, J3.4
- net BUF5_VOUT: now also J19.1, J3.5
- net BUF6_VOUT: now also J17.1, J3.6
- net BUF7_VOUT: now also J15.1, J3.7
- net BUF8_VOUT: now also J13.1, J3.8
- net BUF9_VOUT: now also J11.1, J3.9
- no-connect marks 0 -> 1

Commit message: finished designing new pcb
Parts:
- added J29, J31, J49, J50, J51, J52, J53, J54, J55, J56, J57, J58: Conn_Coaxial, Connector_Coaxial:MMCX_Molex_73415-1471_Vertical, symbol Connector:Conn_Coaxial
Connections:
- net AGND: now also J29.2 (Ext), J31.2 (Ext), J49.2 (Ext), J50.2 (Ext), J51.2 (Ext), J52.2 (Ext), J53.2 (Ext), J54.2 (Ext), J55.2 (Ext), J56.2 (Ext), J57.2 (Ext), J58.2 (Ext)
- new net MARK1_5V: J29.1 (In)
- new net MARK2_5V: J31.1 (In)
- new net MARK3_5V: J49.1 (In)
- new net MARK4_5V: J50.1 (In)
- new net MARK5_5V: J51.1 (In)
- new net MARK6_5V: J52.1 (In)
- new net MARK7_5V: J53.1 (In)
- new net MARK8_5V: J54.1 (In)
- new net TRIG1_5V: J55.1 (In)
- new net TRIG2_5V: J56.1 (In)
- new net TRIG3_5V: J57.1 (In)
- new net TRIG4_5V: J58.1 (In)

Commit message: cleared drc
Parts:
- added J70, J71: RFPC-SMA28-F, dacboard-new:RFPC-SMA28-F, symbol RFPC-SMA28-F:RFPC-SMA28-F
- J10, J11, J12, J13, J14, J15, J16, J17, J18, J19, J20, J21, J22, J32, J33, J34, J35, J36, J4, J5, J6, J7, J8, J9: footprint RFPC-SMA28-F:GRADCONN_RFPC-SMA28-F -> dacboard-new:RFPC-SMA28-F
- J3: footprint DLS3XS6AK44X:CONN_DLS3XS6AK44X_CEC -> dacboard-new:DLS3XS6AK44X
Connections:
- net AGND: now also J70.1, J71.1; no longer J29.2 (Ext), J31.2 (Ext), J49.2 (Ext), J50.2 (Ext), J51.2 (Ext), J52.2 (Ext), J53.2 (Ext), J54.2 (Ext), J55.2 (Ext), J56.2 (Ext), J57.2 (Ext), J58.2 (Ext)
- new net DGND: J29.2 (Ext), J31.2 (Ext), J49.2 (Ext), J50.2 (Ext), J51.2 (Ext), J52.2 (Ext), J53.2 (Ext), J54.2 (Ext), J55.2 (Ext), J56.2 (Ext), J57.2 (Ext), J58.2 (Ext)
- no-connect marks 1 -> 9
