File: pcb/dacboard-new/vita57.4_fmc+.kicad_sch (KiCad schematic)
At the start: 5 parts, among them J27 ASP-184330-01, J28 Conn_02x12_Odd_Even, J29 Conn_02x12_Odd_Even, J30 Conn_02x12_Odd_Even, J31 Conn_02x12_Odd_Even

Commit message: finished designing new pcb
Parts:
- removed J29, J31: Conn_02x12_Odd_Even, Connector_PinHeader_2.54mm:PinHeader_2x12_P2.54mm_Vertical, symbol Connector_Generic:Conn_02x12_Odd_Even
- added J59, J60, J61, J62, J66, J67, J68, J69: Conn_01x02, Connector_PinHeader_2.54mm:PinHeader_1x02_P2.54mm_Vertical, symbol Connector_Generic:Conn_01x02
- added J64, J65: Conn_02x12_Odd_Even, Connector_PinHeader_2.54mm:PinHeader_2x12_P2.54mm_Vertical, symbol Connector_Generic:Conn_02x12_Odd_Even
Connections:
- net ADCIO_00: now also J30.2 (Pin_2); no longer J30.1 (Pin_1)
- net ADCIO_01: now also J30.4 (Pin_4); no longer J30.3 (Pin_3)
- net ADCIO_02: now also J30.8 (Pin_8); no longer J30.7 (Pin_7)
- net ADCIO_03: now also J30.10 (Pin_10); no longer J30.9 (Pin_9)
- net ADCIO_04: now also J30.14 (Pin_14); no longer J30.13 (Pin_13)
- net ADCIO_05: now also J30.16 (Pin_16); no longer J30.15 (Pin_15)
- net ADCIO_06: now also J30.20 (Pin_20); no longer J30.19 (Pin_19)
- net ADCIO_07: now also J30.22 (Pin_22); no longer J30.21 (Pin_21)
- net ADCIO_08: now also J65.2 (Pin_2)
- net ADCIO_09: now also J65.4 (Pin_4)
- net ADCIO_10: now also J30.3 (Pin_3); no longer J30.4 (Pin_4)
- net ADCIO_11: now also J30.5 (Pin_5); no longer J30.6 (Pin_6)
- net ADCIO_12: now also J30.9 (Pin_9); no longer J30.10 (Pin_10)
- net ADCIO_13: now also J30.11 (Pin_11); no longer J30.12 (Pin_12)
- net ADCIO_14: now also J30.15 (Pin_15); no longer J30.16 (Pin_16)
- net ADCIO_15: now also J30.17 (Pin_17); no longer J30.18 (Pin_18)
- net DACIO_00: now also J28.2 (Pin_2); no longer J28.1 (Pin_1)
- net DACIO_01: now also J28.4 (Pin_4); no longer J28.3 (Pin_3)
- net DACIO_03: now also J28.10 (Pin_10); no longer J28.9 (Pin_9)
- net DACIO_04: now also J28.14 (Pin_14); no longer J28.13 (Pin_13)
- net DACIO_05: now also J28.16 (Pin_16); no longer J28.15 (Pin_15)
- net DACIO_06: now also J28.20 (Pin_20); no longer J28.19 (Pin_19)
- net DACIO_07: now also J28.22 (Pin_22); no longer J28.21 (Pin_21)
- net DACIO_08: now also J64.2 (Pin_2)
- net DACIO_09: now also J64.4 (Pin_4)
- net DACIO_10: now also J28.3 (Pin_3); no longer J28.4 (Pin_4)
- net DACIO_12: now also J28.9 (Pin_9); no longer J28.10 (Pin_10)
- net DACIO_13: now also J28.11 (Pin_11); no longer J28.12 (Pin_12)
- net DACIO_14: now also J28.15 (Pin_15); no longer J28.16 (Pin_16)
- net E39_VADJ: now also J59.2 (Pin_2)
- net F40_VADJ: now also J60.2 (Pin_2)
- net G39_VADJ: now also J61.2 (Pin_2)
- net H40_VADJ: now also J62.2 (Pin_2)
- net VCCN: now also J59.1 (Pin_1), J60.1 (Pin_1), J61.1 (Pin_1), J62.1 (Pin_1), J66.1 (Pin_1), J67.1 (Pin_1), J68.1 (Pin_1), J69.1 (Pin_1)
- net D15_LA09_N renamed CS_N_CH16
- net D21_LA17_N_CC renamed CS_N_CH20
- net D27_LA26_N renamed CS_N_CH9
- net D8_LA01_P_CC renamed CS_N_CH3
- net D9_LA01_N_CC renamed CS_N_CH15
- net DACIO_02: no longer names the net of J28.7 (Pin_7)
- net DACIO_11: no longer names the net of J28.6 (Pin_6)
- net DACIO_15: no longer names the net of J28.18 (Pin_18)
- net G12_LA08_P renamed CS_N_CH18
- net G21_LA20_P renamed CS_N_CH8
- net G25_LA22_N renamed CS_N_CH7
- net G28_LA25_N renamed CS_N_CH21
- net G34_LA31_N renamed CS_N_CH22
- net H11_LA04_N renamed CS_N_CH6
- net H16_LA11_P renamed CS_N_CH17
- net H17_LA11_N renamed CS_N_CH5
- net H26_LA21_N renamed CS_N_CH19
- net H34_LA30_P renamed CS_N_CH10
- removed net NGND: J28.11 (Pin_11), J28.14 (Pin_14), J28.17 (Pin_17), J28.2 (Pin_2), J28.20 (Pin_20), J28.23 (Pin_23), J28.5 (Pin_5), J28.8 (Pin_8), J30.11 (Pin_11), J30.14 (Pin_14), J30.17 (Pin_17), J30.2 (Pin_2), J30.20 (Pin_20), J30.23 (Pin_23), J30.5 (Pin_5), J30.8 (Pin_8)
- net SYNC_C2M_N renamed LDAC_N_CH2
- net SYNC_C2M_P renamed MOSI_CH2
- net SYNC_M2C_N renamed SCLK_CH11
- net SYNC_M2C_P renamed CS_N_CH11
- new net CS_N_CH12: J28.8 (Pin_8)
- new net CS_N_CH23: J28.17 (Pin_17)
- new net CS_N_CH24: J28.5 (Pin_5)
- new net VADJ_ADC: J65.14 (Pin_14), J65.16 (Pin_16), J67.2 (Pin_2), J69.2 (Pin_2)
- new net VADJ_DAC: J64.10 (Pin_10), J64.12 (Pin_12), J66.2 (Pin_2), J68.2 (Pin_2)
- no-connect marks 231 -> 410

Commit message: cleared drc
Connections:
- net C30_SCL: no longer names the net of J27.C30
- net C31_SDA: no longer names the net of J27.C31
- net C34_GA0: no longer names the net of J27.C34
- net C35_12P0V: no longer names the net of J27.C35
- net C37_12P0V: no longer names the net of J27.C37
- net C39_3P3V: no longer names the net of J27.C39
- net D1_PG_C2M: no longer names the net of J27.D01
- net D29_TCK: no longer names the net of J27.D29
- net D30_TDI: no longer names the net of J27.D30
- net D31_TDO: no longer names the net of J27.D31
- net D32_3P3VAUX: no longer names the net of J27.D32
- net D33_TMS: no longer names the net of J27.D33
- net D35_GA1: no longer names the net of J27.D35
- net D36_3P3V: no longer names the net of J27.D36
- net D38_3P3V: no longer names the net of J27.D38
- net D40_3P3V: no longer names the net of J27.D40
- net DP0_C2M_N: no longer names the net of J27.C03
- net DP0_C2M_P: no longer names the net of J27.C02
- net DP0_M2C_N: no longer names the net of J27.C07
- net DP0_M2C_P: no longer names the net of J27.C06
- net DP1_C2M_N: no longer names the net of J27.A23
- net DP1_C2M_P: no longer names the net of J27.A22
- net DP1_M2C_N: no longer names the net of J27.A03
- net DP1_M2C_P: no longer names the net of J27.A02
- net DP2_C2M_N: no longer names the net of J27.A27
- net DP2_C2M_P: no longer names the net of J27.A26
- net DP2_M2C_N: no longer names the net of J27.A07
- net DP2_M2C_P: no longer names the net of J27.A06
- net DP3_C2M_N: no longer names the net of J27.A31
- net DP3_C2M_P: no longer names the net of J27.A30
- net DP3_M2C_N: no longer names the net of J27.A11
- net DP3_M2C_P: no longer names the net of J27.A10
- net DP4_C2M_N: no longer names the net of J27.A35
- net DP4_C2M_P: no longer names the net of J27.A34
- net DP4_M2C_N: no longer names the net of J27.A15
- net DP4_M2C_P: no longer names the net of J27.A14
- net DP5_C2M_N: no longer names the net of J27.A39
- net DP5_C2M_P: no longer names the net of J27.A38
- net DP5_M2C_N: no longer names the net of J27.A19
- net DP5_M2C_P: no longer names the net of J27.A18
- net DP6_C2M_N: no longer names the net of J27.B37
- net DP6_C2M_P: no longer names the net of J27.B36
- net DP6_M2C_N: no longer names the net of J27.B17
- net DP6_M2C_P: no longer names the net of J27.B16
- net DP7_C2M_N: no longer names the net of J27.B33
- net DP7_C2M_P: no longer names the net of J27.B32
- net DP7_M2C_N: no longer names the net of J27.B13
- net DP7_M2C_P: no longer names the net of J27.B12
- net F1_PG_M2C: no longer names the net of J27.F01
- net GBTCLK0_M2C_N: no longer names the net of J27.D05
- net GBTCLK0_M2C_P: no longer names the net of J27.D04
- net GBTCLK1_M2C_N: no longer names the net of J27.B21
- net GBTCLK1_M2C_P: no longer names the net of J27.B20
- removed net GND: J27.B03, J27.B06, J27.B10, J27.B11, J27.B23, J27.B27, J27.B31, J27.C16, J27.C17, J27.C36, J27.C38, J27.C40, J27.D03, J27.D06, J27.D16, J27.D37, J27.E01, J27.E04, J27.E05, J27.E08, J27.E11, J27.E20, J27.E38, J27.E40, J27.F09, J27.F12, J27.F18, J27.F39, J27.G01, J27.G08, J27.G11, J27.G14, J27.G17, J27.G20, J27.G23, J27.G32, J27.G35, J27.G38, J27.H03, J27.H39, J27.J04, J27.J05, J27.J17, J27.J38, J27.J40, J27.K02, J27.K03, J27.K24, J27.K27, J27.L02, J27.L03, J27.L19, J27.M01, J27.M04, J27.M05, J27.M16, J27.M40, J27.Y01, J27.Y04, J27.Y05, J27.Y40, J27.Z34
- net H1_VREF_A_M2C: no longer names the net of J27.H01
- net H2_PRSNT_M2C_L: no longer names the net of J27.H02
- net J39_VIO_B_M2C: no longer names the net of J27.J39
- net K1_VREF_B_M2C: no longer names the net of J27.K01
- net K40_VIO_B_M2C: no longer names the net of J27.K40
- net L36_12P0V: no longer names the net of J27.L36
- net L37_12P0V: no longer names the net of J27.L37
- net L40_12P0V: no longer names the net of J27.L40
- net REFCLK_C2M_N: no longer names the net of J27.L21
- net REFCLK_C2M_P: no longer names the net of J27.L20
- net REFCLK_M2C_N: no longer names the net of J27.L25
- net REFCLK_M2C_P: no longer names the net of J27.L24
- net VADJ_ADC renamed VADJ_ADC1
- net VADJ_ADC1: no longer J65.16 (Pin_16), J69.2 (Pin_2)
- net VADJ_DAC renamed VADJ_DAC1
- net VADJ_DAC1: no longer J64.12 (Pin_12), J68.2 (Pin_2)
- net Z1_HSPC_PRSNT_M2C_L: no longer names the net of J27.Z01
- net Z40_3P3V: no longer names the net of J27.Z40
- new net NGND: J27.E11, J27.E20, J27.F12, J27.F18, J27.G01, J27.G14, J27.G17, J27.G20, J27.G23, J27.H03, J27.J04, J27.J05, J27.J38, J27.J40, J27.K02, J27.K03, J27.K24, J27.L02, J27.L03, J27.L19, J27.M01, J27.M04, J27.M05, J27.M16, J27.M40
- new net VADJ_ADC2: J65.16 (Pin_16), J69.2 (Pin_2)
- new net VADJ_DAC2: J64.12 (Pin_12), J68.2 (Pin_2)
- no-connect marks 410 -> 513
